File: pcb/2chop.sch (KiCad schematic (older format))
At the start: 26 parts, among them K301 CONN_3, K302 CONN_3, P301 CONN_5X2, U301 TL082

Commit message: städa lite
Parts:
- R302, R305, R309: value 0 -> 0R
- R307, R314: value 10 -> 10R
Connections:
- net AGND: now also P301.2, P301.4, P301.6, P301.8
Other:
- moved on the sheet: C501, C502, C503, C504, C505, C506, C507, C508, K501, K502, P501, R501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

Commit message: fuffens
Changed lines of the file:
@@
-EESchema Schematic File Version 2  date Tue 02 Apr 2013 02:02:16 PM CEST
+EESchema Schematic File Version 2  date Tue 02 Apr 2013 03:24:17 PM CEST
 LIBS:power
 LIBS:device
@@
 $Descr A4 11693 8268
 encoding utf-8
-Sheet 5 6
+Sheet 4 6
 Title "radaq"
 Date "2 apr 2013"
@@
 AR Path="/5152811C/5141E5EA" Ref="U501"  Part="1"
 AR Path="/51529554/5141E5EA" Ref="U601"  Part="1"
-F 0 "U501" H 4500 4150 60  0000 L CNN
+F 0 "U401" H 4500 4150 60  0000 L CNN
 F 1 "TL082" H 4500 3700 60  0000 L CNN
 F 2 "" H 4550 3950 60  0001 C CNN
@@
 AR Path="/5152811C/5141E658" Ref="R506"  Part="1"
 AR Path="/51529554/5141E658" Ref="R606"  Part="1"
-F 0 "R506" V 4880 3200 50  0000 C CNN
+F 0 "R406" V 4880 3200 50  0000 C CNN
 F 1 "1K" V 4800 3200 50  0000 C CNN
 F 2 "" H 4800 3200 60  0001 C CNN
@@
 AR Path="/5152811C/5141E665" Ref="R503"  Part="1"
 AR Path="/51529554/5141E665" Ref="R603"  Part="1"
-F 0 "R503" V 3480 3200 50  0000 C CNN
+F 0 "R403" V 3480 3200 50  0000 C CNN
 F 1 "NI" V 3400 3200 50  0000 C CNN
 F 2 "" H 3400 3200 60  0001 C CNN
@@
 AR Path="/5152811C/5141E66B" Ref="R504"  Part="1"
 AR Path="/51529554/5141E66B" Ref="R604"  Part="1"
-F 0 "R504" V 3480 3850 50  0000 C CNN
+F 0 "R404" V 3480 3850 50  0000 C CNN
 F 1 "1K" V 3400 3850 50  0000 C CNN
 F 2 "" H 3400 3850 60  0001 C CNN
@@
 AR Path="/5152811C/5141E671" Ref="R505"  Part="1"
 AR Path="/51529554/5141E671" Ref="R605"  Part="1"
-F 0 "R505" V 3480 4050 50  0000 C CNN
+F 0 "R405" V 3480 4050 50  0000 C CNN
 F 1 "0R" V 3400 4050 50  0000 C CNN
 F 2 "" H 3400 4050 60  0001 C CNN
@@
 AR Path="/5152811C/5141E677" Ref="R502"  Part="1"
 AR Path="/51529554/5141E677" Ref="R602"  Part="1"
-F 0 "R502" H 2950 4300 50  0000 C CNN
+F 0 "R402" H 2950 4300 50  0000 C CNN
 F 1 "0R" V 3150 4400 50  0000 C CNN
 F 2 "" H 3150 4400 60  0001 C CNN
@@
 AR Path="/5152811C/5141E67D" Ref="R501"  Part="1"
 AR Path="/51529554/5141E67D" Ref="R601"  Part="1"
-F 0 "R501" V 2750 4050 50  0000 C CNN
+F 0 "R401" V 2750 4050 50  0000 C CNN
 F 1 "NI" V 2650 4050 50  0000 C CNN
 F 2 "" H 2650 4050 60  0001 C CNN
@@
 AR Path="/5152811C/515177F5" Ref="C501"  Part="1"
 AR Path="/51529554/515177F5" Ref="C601"  Part="1"
-F 0 "C501" H 2700 4500 50  0000 L CNN
+F 0 "C401" H 2700 4500 50  0000 L CNN
 F 1 "NI" H 2800 4300 50  0000 L CNN
 F 2 "" H 2900 4400 60  0001 C CNN
@@
 AR Path="/5152811C/51517804" Ref="C504"  Part="1"
 AR Path="/51529554/51517804" Ref="C604"  Part="1"
-F 0 "C504" V 4900 3450 50  0000 L CNN
+F 0 "C404" V 4900 3450 50  0000 L CNN
 F 1 "39pF" V 4800 3450 50  0000 L CNN
 F 2 "" H 4850 3400 60  0001 C CNN
@@
 AR Path="/5152811C/5151790E" Ref="R513"  Part="1"
 AR Path="/51529554/5151790E" Ref="R613"  Part="1"
-F 0 "R513" V 8630 3200 50  0000 C CNN
+F 0 "R413" V 8630 3200 50  0000 C CNN
 F 1 "1K" V 8550 3200 50  0000 C CNN
 F 2 "" H 8550 3200 60  0001 C CNN
@@
 AR Path="/5152811C/51517914" Ref="R510"  Part="1"
 AR Path="/51529554/51517914" Ref="R610"  Part="1"
-F 0 "R510" V 7230 3200 50  0000 C CNN
+F 0 "R410" V 7230 3200 50  0000 C CNN
 F 1 "NI" V 7150 3200 50  0000 C CNN
 F 2 "" H 7150 3200 60  0001 C CNN
@@
 AR Path="/5152811C/5151791A" Ref="R511"  Part="1"
 AR Path="/51529554/5151791A" Ref="R611"  Part="1"
-F 0 "R511" V 7230 3850 50  0000 C CNN
+F 0 "R411" V 7230 3850 50  0000 C CNN
 F 1 "1K" V 7150 3850 50  0000 C CNN
 F 2 "" H 7150 3850 60  0001 C CNN
@@
 AR Path="/5152811C/51517920" Ref="R512"  Part="1"
 AR Path="/51529554/51517920" Ref="R612"  Part="1"
-F 0 "R512" V 7230 4050 50  0000 C CNN
+F 0 "R412" V 7230 4050 50  0000 C CNN
 F 1 "0" V 7150 4050 50  0000 C CNN
 F 2 "" H 7150 4050 60  0001 C CNN
@@
 AR Path="/5152811C/51517926" Ref="R509"  Part="1"
 AR Path="/51529554/51517926" Ref="R609"  Part="1"
-F 0 "R509" H 6700 4350 50  0000 C CNN
+F 0 "R409" H 6700 4350 50  0000 C CNN
 F 1 "0R" V 6900 4400 50  0000 C CNN
 F 2 "" H 6900 4400 60  0001 C CNN
@@
 AR Path="/5152811C/5151792C" Ref="R508"  Part="1"
 AR Path="/51529554/5151792C" Ref="R608"  Part="1"
-F 0 "R508" V 6500 4050 50  0000 C CNN
+F 0 "R408" V 6500 4050 50  0000 C CNN
 F 1 "NI" V 6400 4050 50  0000 C CNN
 F 2 "" H 6400 4050 60  0001 C CNN
@@
 AR Path="/5152811C/51517941" Ref="C506"  Part="1"
 AR Path="/51529554/51517941" Ref="C606"  Part="1"
-F 0 "C506" H 6450 4500 50  0000 L CNN
+F 0 "C406" H 6450 4500 50  0000 L CNN
 F 1 "NI" H 6550 4300 50  0000 L CNN
 F 2 "" H 6650 4400 60  0001 C CNN
@@
 AR Path="/5152811C/51517947" Ref="C507"  Part="1"
 AR Path="/51529554/51517947" Ref="C607"  Part="1"
-F 0 "C507" V 8650 3450 50  0000 L CNN
+F 0 "C407" V 8650 3450 50  0000 L CNN
 F 1 "39pF" V 8550 3450 50  0000 L CNN
 F 2 "" H 8600 3400 60  0001 C CNN
@@
 AR Path="/5152811C/5141E5BD" Ref="U501"  Part="2"
 AR Path="/51529554/5141E5BD" Ref="U601"  Part="2"
-F 0 "U501" H 8250 4150 60  0000 L CNN
+F 0 "U401" H 8250 4150 60  0000 L CNN
 F 1 "TL082" H 8250 3700 60  0000 L CNN
 F 2 "" H 8300 3950 60  0001 C CNN
@@
 AR Path="/5152811C/5151B311" Ref="C502"  Part="1"
 AR Path="/51529554/5151B311" Ref="C602"  Part="1"
-F 0 "C502" H 2950 1850 50  0000 L CNN
+F 0 "C402" H 2950 1850 50  0000 L CNN
 F 1 "100nF" H 2950 1950 50  0000 L CNN
 F 2 "" H 2800 1900 60  0001 C CNN
@@
 AR Path="/5152811C/5151B335" Ref="C503"  Part="1"
 AR Path="/51529554/5151B335" Ref="C603"  Part="1"
-F 0 "C503" H 2750 1850 50  0000 L CNN
+F 0 "C403" H 2750 1850 50  0000 L CNN
 F 1 "100nF" H 2700 1950 50  0000 L CNN
 F 2 "" H 3100 1900 60  0001 C CNN
@@
 AR Path="/5152811C/515217D1" Ref="R507"  Part="1"
 AR Path="/51529554/515217D1" Ref="R607"  Part="1"
-F 0 "R507" V 5680 4300 50  0000 C CNN
+F 0 "R407" V 5680 4300 50  0000 C CNN
 F 1 "10R" V 5600 4300 50  0000 C CNN
 F 2 "" H 5600 4300 60  0001 C CNN
@@
 AR Path="/5152811C/515217E3" Ref="C505"  Part="1"
 AR Path="/51529554/515217E3" Ref="C605"  Part="1"
-F 0 "C505" H 6000 4450 50  0000 L CNN
+F 0 "C405" H 6000 4450 50  0000 L CNN
 F 1 "2200pF" H 6000 4550 50  0000 L CNN
 F 2 "" H 5850 4500 60  0001 C CNN
@@
 AR Path="/5152811C/51521807" Ref="#PWR053"  Part="1"
 AR Path="/51529554/51521807" Ref="#PWR062"  Part="1"
-F 0 "#PWR053" H 3150 3300 40  0001 C CNN
+F 0 "#PWR044" H 3150 3300 40  0001 C CNN
 F 1 "AGND" H 3150 3230 50  0000 C CNN
 F 2 "" H 3150 3300 60  0001 C CNN
@@
 AR Path="/5152811C/5152181E" Ref="#PWR054"  Part="1"
 AR Path="/51529554/5152181E" Ref="#PWR063"  Part="1"
-F 0 "#PWR054" H 3150 4750 40  0001 C CNN
+F 0 "#PWR045" H 3150 4750 40  0001 C CNN
 F 1 "AGND" H 3150 4680 50  0000 C CNN
 F 2 "" H 3150 4750 60  0001 C CNN
@@
 AR Path="/5152811C/51521824" Ref="#PWR055"  Part="1"
 AR Path="/51529554/51521824" Ref="#PWR064"  Part="1"
-F 0 "#PWR055" H 2950 2250 40  0001 C CNN
+F 0 "#PWR046" H 2950 2250 40  0001 C CNN
 F 1 "AGND" H 2950 2180 50  0000 C CNN
 F 2 "" H 2950 2250 60  0001 C CNN
@@
 AR Path="/5152811C/5152182A" Ref="#PWR056"  Part="1"
 AR Path="/51529554/5152182A" Ref="#PWR065"  Part="1"
-F 0 "#PWR056" H 6900 4750 40  0001 C CNN
+F 0 "#PWR047" H 6900 4750 40  0001 C CNN
 F 1 "AGND" H 6900 4680 50  0000 C CNN
 F 2 "" H 6900 4750 60  0001 C CNN
@@
 AR Path="/5152811C/5152183A" Ref="#PWR057"  Part="1"
 AR Path="/51529554/5152183A" Ref="#PWR066"  Part="1"
-F 0 "#PWR057" H 5850 4800 40  0001 C CNN
+F 0 "#PWR048" H 5850 4800 40  0001 C CNN
 F 1 "AGND" H 5850 4730 50  0000 C CNN
 F 2 "" H 5850 4800 60  0001 C CNN
@@
 AR Path="/5152811C/5152184A" Ref="#PWR058"  Part="1"
 AR Path="/51529554/5152184A" Ref="#PWR067"  Part="1"
-F 0 "#PWR058" H 6900 3300 40  0001 C CNN
+F 0 "#PWR049" H 6900 3300 40  0001 C CNN
 F 1 "AGND" H 6900 3230 50  0000 C CNN
 F 2 "" H 6900 3300 60  0001 C CNN
@@
 AR Path="/5152811C/5152185C" Ref="R514"  Part="1"
 AR Path="/51529554/5152185C" Ref="R614"  Part="1"
-F 0 "R514" V 9480 4300 50  0000 C CNN
+F 0 "R414" V 9480 4300 50  0000 C CNN
 F 1 "10R" V 9400 4300 50  0000 C CNN
 F 2 "" H 9400 4300 60  0001 C CNN
@@
 AR Path="/5152811C/51521862" Ref="C508"  Part="1"
 AR Path="/51529554/51521862" Ref="C608"  Part="1"
-F 0 "C508" H 9800 4450 50  0000 L CNN
+F 0 "C408" H 9800 4450 50  0000 L CNN
 F 1 "2200pF" H 9800 4550 50  0000 L CNN
 F 2 "" H 9650 4500 60  0001 C CNN
@@
 AR Path="/5152811C/5152186E" Ref="#PWR059"  Part="1"
 AR Path="/51529554/5152186E" Ref="#PWR068"  Part="1"
-F 0 "#PWR059" H 9650 4800 40  0001 C CNN
+F 0 "#PWR050" H 9650 4800 40  0001 C CNN
 F 1 "AGND" H 9650 4730 50  0000 C CNN
 F 2 "" H 9650 4800 60  0001 C CNN
@@
 AR Path="/5152811C/5152197F" Ref="K502"  Part="1"
 AR Path="/51529554/5152197F" Ref="K602"  Part="1"
-F 0 "K502" V 9100 3600 50  0000 C CNN
+F 0 "K402" V 9100 3600 50  0000 C CNN
 F 1 "CONN_3" V 9200 3600 40  0000 C CNN
 F 2 "" H 9150 3600 60  0001 C CNN
@@
 AR Path="/5152811C/51521A30" Ref="K501"  Part="1"
 AR Path="/51529554/51521A30" Ref="K601"  Part="1"
-F 0 "K501" V 5300 3600 50  0000 C CNN
+F 0 "K401" V 5300 3600 50  0000 C CNN
 F 1 "CONN_3" V 5400 3600 40  0000 C CNN
 F 2 "" H 5350 3600 60  0001 C CNN
@@
 AR Path="/5152811C/515254E2" Ref="P501"  Part="1"
 AR Path="/51529554/515254E2" Ref="P601"  Part="1"
-F 0 "P501" H 4500 2200 60  0000 C CNN
+F 0 "P401" H 4500 2200 60  0000 C CNN
 F 1 "CONN_5X2" V 4500 1900 50  0000 C CNN
 F 2 "" H 4500 1900 60  0001 C CNN
@@
 AR Path="/5152811C/515254EF" Ref="#PWR061"  Part="1"
 AR Path="/51529554/515254EF" Ref="#PWR070"  Part="1"
-F 0 "#PWR061" H 4150 1500 40  0001 C CNN
+F 0 "#PWR052" H 4150 1500 40  0001 C CNN
 F 1 "AGND" H 4150 1430 50  0000 C CNN
 F 2 "" H 4150 1500 60  0001 C CNN
