File: pcb/power.sch (KiCad schematic (older format))
At the start: 14 parts, among them U201 LT3032, U202 IA0515S_

Commit message: städa lite
Other:
- moved on the sheet: C208, RV201, RV202
Changed lines of the file:
@@
-EESchema Schematic File Version 2  date Mon 01 Apr 2013 04:53:06 PM CEST
+EESchema Schematic File Version 2  date Tue 02 Apr 2013 02:02:16 PM CEST
 LIBS:power
 LIBS:device
@@
 LIBS:contrib
 LIBS:valves
-LIBS:raspi
-LIBS:ti
-LIBS:ia0515s_
-LIBS:lt3032
-LIBS:bq32000
 LIBS:curry2-cache
 EELAYER 27 0
@@
 encoding utf-8
 Sheet 2 6
-Title ""
-Date "1 apr 2013"
-Rev ""
+Title "radaq"
+Date "2 apr 2013"
+Rev "R1A"
 Comp ""
 Comment1 ""
@@
 $EndComp
 $Comp
-L LT3032 U201
-U 1 1 5151B8CC
-P 5800 3450
-F 0 "U201" H 5800 3700 60  0000 C CNN
-F 1 "LT3032" H 5800 3800 60  0000 C CNN
-F 2 "" H 5800 3450 60  0001 C CNN
-F 3 "" H 5800 3450 60  0001 C CNN
-	1    5800 3450
-	1    0    0    -1
-$EndComp
-$Comp
 L C C205
 U 1 1 5151BA9D
 P 4300 3400
-F 0 "C205" H 4350 3500 50  0000 L CNN
-F 1 "C" H 4350 3300 50  0000 L CNN
+F 0 "C205" V 4250 3450 50  0000 L CNN
+F 1 "C" V 4350 3450 50  0000 L CNN
 F 2 "" H 4300 3400 60  0001 C CNN
 F 3 "" H 4300 3400 60  0001 C CNN
@@
 U 1 1 5151BAAC
 P 5050 4100
-F 0 "C206" H 5100 4200 50  0000 L CNN
-F 1 "C" H 5100 4000 50  0000 L CNN
+F 0 "C206" H 4650 4000 50  0000 L CNN
+F 1 "C" H 4800 4100 50  0000 L CNN
 F 2 "" H 5050 4100 60  0001 C CNN
 F 3 "" H 5050 4100 60  0001 C CNN
@@
 L POT RV202
 U 1 1 5151EBB9
-P 6300 4350
-F 0 "RV202" H 6300 4250 50  0000 C CNN
-F 1 "POT" H 6300 4350 50  0000 C CNN
-F 2 "" H 6300 4350 60  0001 C CNN
-F 3 "" H 6300 4350 60  0001 C CNN
-	1    6300 4350
+P 6600 4150
+F 0 "RV202" H 6600 4050 50  0000 C CNN
+F 1 "POT" H 6600 4150 50  0000 C CNN
+F 2 "" H 6600 4150 60  0001 C CNN
+F 3 "" H 6600 4150 60  0001 C CNN
+	1    6600 4150
 	1    0    0    -1
 $EndComp
@@
 L POT RV201
 U 1 1 5151EC34
-P 4800 3300
-F 0 "RV201" H 4800 3200 50  0000 C CNN
-F 1 "POT" H 4800 3300 50  0000 C CNN
-F 2 "" H 4800 3300 60  0001 C CNN
-F 3 "" H 4800 3300 60  0001 C CNN
-	1    4800 3300
-	0    1    1    0
-$EndComp
-Text HLabel 6800 3400 2    60   Input ~ 0
+P 4700 2900
+F 0 "RV201" H 4700 2800 50  0000 C CNN
+F 1 "POT" H 4700 2900 50  0000 C CNN
+F 2 "" H 4700 2900 60  0001 C CNN
+F 3 "" H 4700 2900 60  0001 C CNN
+	1    4700 2900
+	-1   0    0    1
+$EndComp
+Text HLabel 6900 3400 2    60   Input ~ 0
 Enable
 Wire Wire Line
-	3750 3200 5050 3200
+	3750 3200 3900 3200
+Wire Wire Line
+	3900 3200 4100 3200
+Wire Wire Line
+	4100 3200 4950 3200
+Wire Wire Line
+	4950 3200 5050 3200
 Wire Wire Line
 	5050 3800 5050 3900
 Wire Wire Line
-	5050 4300 5050 4450
-Wire Wire Line
-	5050 4450 7200 4450
-Wire Wire Line
-	7200 4450 7200 3500
-Wire Wire Line
-	7200 3500 6600 3500
-Wire Wire Line
-	6050 4350 5250 4350
-Wire Wire Line
-	5250 4350 5250 3900
-Wire Wire Line
-	5250 3900 5050 3900
-Wire Wire Line
-	6300 4200 6300 4000
-Wire Wire Line
-	6300 4000 6600 4000
+	5050 4300 5050 4500
+Wire Wire Line
+	5050 4500 7000 4500
+Wire Wire Line
+	7000 4500 7000 3500
+Wire Wire Line
+	7000 3500 6600 3500
+Wire Wire Line
+	5200 4400 5200 3900
+Wire Wire Line
+	5200 3900 5050 3900
+Wire Wire Line
+	6600 4000 6600 4000
 Wire Wire Line
 	6600 4000 6600 3800
 Wire Wire Line
-	6550 4350 6550 4400
+	6850 4150 6850 4250
 Wire Wire Line
 	5700 4200 5700 4250
 Wire Wire Line
-	5050 3300 4950 3300
-Wire Wire Line
-	4800 3050 4950 3050
-Wire Wire Line
-	4950 3050 4950 3200
+	5050 3300 4700 3300
+Wire Wire Line
+	4950 2900 4950 3200
 Connection ~ 4950 3200
 Wire Wire Line
@@
 	6800 3600 6800 3400
 Wire Wire Line
-	6800 3400 6600 3400
+	6600 3400 6800 3400
+Wire Wire Line
+	6800 3400 6900 3400
 Wire Wire Line
 	8050 3200 8050 3950
 Wire Wire Line
-	6600 3200 8050 3200
-Wire Wire Line
-	8050 4250 7550 4250
-Wire Wire Line
-	7550 4600 7550 3700
-Wire Wire Line
-	7550 3700 6600 3700
-Wire Wire Line
-	5050 3700 4850 3700
-Wire Wire Line
-	4850 3700 4850 4600
-Wire Wire Line
-	4850 4600 7550 4600
-Connection ~ 7550 4250
+	6600 3200 7650 3200
+Wire Wire Line
+	7650 3200 8050 3200
+Wire Wire Line
+	8050 4250 7100 4250
+Wire Wire Line
+	7100 4600 7100 4250
+Wire Wire Line
+	7100 4250 7100 3700
+Wire Wire Line
+	7100 3700 6600 3700
+Wire Wire Line
+	5050 3700 4900 3700
+Wire Wire Line
+	4900 3700 4900 4600
+Wire Wire Line
+	4900 4600 5800 4600
+Wire Wire Line
+	5800 4600 7000 4600
+Wire Wire Line
+	7000 4600 7100 4600
+Connection ~ 7100 4250
 Wire Wire Line
 	5800 4200 5800 4600
@@
 $EndComp
 Wire Wire Line
-	5050 3800 3750 3800
+	3750 3800 3900 3800
+Wire Wire Line
+	3900 3800 5050 3800
 Wire Wire Line
 	5050 3400 4500 3400
@@
 $EndComp
 Wire Wire Line
-	3150 3200 2900 3200
+	2800 3200 2900 3200
+Wire Wire Line
+	2900 3200 3150 3200
 Wire Wire Line
 	2900 3600 2900 3650
 Wire Wire Line
-	3150 3800 2900 3800
+	2800 3800 2900 3800
+Wire Wire Line
+	2900 3800 3150 3800
 Wire Wire Line
 	2900 4200 2900 4300
@@
 L C C208
 U 1 1 5151EEE9
-P 7800 3400
-F 0 "C208" H 7850 3500 50  0000 L CNN
-F 1 "C" H 7850 3300 50  0000 L CNN
-F 2 "" H 7800 3400 60  0001 C CNN
-F 3 "" H 7800 3400 60  0001 C CNN
-	1    7800 3400
+P 7650 3400
+F 0 "C208" H 7700 3500 50  0000 L CNN
+F 1 "C" H 7700 3300 50  0000 L CNN
+F 2 "" H 7650 3400 60  0001 C CNN
+F 3 "" H 7650 3400 60  0001 C CNN
+	1    7650 3400
 	-1   0    0    1
 $EndComp
@@
 $EndComp
 Wire Wire Line
-	5050 3500 5050 3600
-Wire Wire Line
 	4550 3700 4550 3600
-Wire Wire Line
-	4550 3600 5050 3600
-Text HLabel 2900 3200 0    60   Input ~ 0
+Text HLabel 2800 3200 0    60   Input ~ 0
 +14
-Text HLabel 2900 3800 0    60   Input ~ 0
+Text HLabel 2800 3800 0    60   Input ~ 0
 -14
 $Comp
@@
 U 1 1 5151F0BF
 P 3900 3400
-F 0 "C203" H 3950 3500 50  0000 L CNN
-F 1 "C" H 3950 3300 50  0000 L CNN
+F 0 "C203" H 3650 3500 50  0000 L CNN
+F 1 "C" H 3800 3300 50  0000 L CNN
 F 2 "" H 3900 3400 60  0001 C CNN
 F 3 "" H 3900 3400 60  0001 C CNN
@@
 U 1 1 5151F0C5
 P 3900 4000
-F 0 "C204" H 3950 4100 50  0000 L CNN
-F 1 "C" H 3950 3900 50  0000 L CNN
+F 0 "C204" H 3650 4100 50  0000 L CNN
+F 1 "C" H 3800 3900 50  0000 L CNN
 F 2 "" H 3900 4000 60  0001 C CNN
 F 3 "" H 3900 4000 60  0001 C CNN
@@
 	3900 4200 3900 4300
 Wire Wire Line
-	7800 3600 7800 3750
+	7650 3600 7650 3700
 Wire Wire Line
 	7000 5000 7000 5050
-Connection ~ 7800 3200
+Connection ~ 7650 3200
 Connection ~ 7000 4600
 $Comp
@@
 L AGND #PWR024
 U 1 1 515849A0
-P 7800 3750
-F 0 "#PWR024" H 7800 3750 40  0001 C CNN
-F 1 "AGND" H 7800 3680 50  0000 C CNN
-F 2 "" H 7800 3750 60  0000 C CNN
-F 3 "" H 7800 3750 60  0000 C CNN
-	1    7800 3750
+P 7650 3700
+F 0 "#PWR024" H 7650 3700 40  0001 C CNN
+F 1 "AGND" H 7650 3630 50  0000 C CNN
+F 2 "" H 7650 3700 60  0000 C CNN
+F 3 "" H 7650 3700 60  0000 C CNN
+	1    7650 3700
 	1    0    0    -1
 $EndComp
@@
 L AGND #PWR026
 U 1 1 515849B6
-P 6550 4400
-F 0 "#PWR026" H 6550 4400 40  0001 C CNN
-F 1 "AGND" H 6550 4330 50  0000 C CNN
-F 2 "" H 6550 4400 60  0000 C CNN
-F 3 "" H 6550 4400 60  0000 C CNN
-	1    6550 4400
+P 6850 4250
+F 0 "#PWR026" H 6850 4250 40  0001 C CNN
+F 1 "AGND" H 6850 4180 50  0000 C CNN
+F 2 "" H 6850 4250 60  0000 C CNN
+F 3 "" H 6850 4250 60  0000 C CNN
+	1    6850 4250
 	1    0    0    -1
 $EndComp
@@
 L AGND #PWR028
 U 1 1 515849C2
-P 4800 3650
-F 0 "#PWR028" H 4800 3650 40  0001 C CNN
-F 1 "AGND" H 4800 3580 50  0000 C CNN
-F 2 "" H 4800 3650 60  0000 C CNN
-F 3 "" H 4800 3650 60  0000 C CNN
-	1    4800 3650
+P 4400 3000
+F 0 "#PWR028" H 4400 3000 40  0001 C CNN
+F 1 "AGND" H 4400 2930 50  0000 C CNN
+F 2 "" H 4400 3000 60  0000 C CNN
+F 3 "" H 4400 3000 60  0000 C CNN
+	1    4400 3000
 	1    0    0    -1
 $EndComp
@@
 	7850 5050 7850 5100
 Wire Wire Line
-	4800 3550 4800 3650
+	4400 2900 4400 3000
 Connection ~ 3900 3200
-Connection ~ 3950 3800
 Connection ~ 2900 3200
 Connection ~ 2900 3800
 Connection ~ 3900 3800
+Wire Wire Line
+	4700 3300 4700 3050
+Wire Wire Line
+	4400 2900 4450 2900
+$Comp
+L LT3032 U201
+U 1 1 5151B8CC
+P 5800 3450
+F 0 "U201" H 5800 3700 60  0000 C CNN
+F 1 "LT3032" H 5800 3800 60  0000 C CNN
+F 2 "" H 5800 3450 60  0001 C CNN
+F 3 "" H 5800 3450 60  0001 C CNN
+	1    5800 3450
+	1    0    0    -1
+$EndComp
+Wire Wire Line
+	6350 4150 6350 4400
+Wire Wire Line
+	6350 4400 5200 4400
+Wire Wire Line
+	5050 3500 5050 3600
+Wire Wire Line
+	5050 3600 4550 3600
+Connection ~ 5050 3600
+Connection ~ 5050 3900
+Connection ~ 6800 3400
 $EndSCHEMATC
