File: pcb/power.sch (KiCad schematic (older format))
At the start: 14 parts, among them U201 LT3032, U202 IA0515S_

Commit message: almost done
Connections:
- net GND: no longer C201.2, C202.2, C203.2, C204.2, C207.1, C208.1, RV201.3, RV202.3, U201.15 (GND), U201.4 (GND), U201.5 (GND), U202.4 (OUTGND)
- net at U201.16 (INN), U201.6 (INN), U201.9 (INN)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: now also C207.2
- net at U201.14 (INP), U202.5 (VOUT+): now also C208.2
- net at C205.2, L201.2, RV201.1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: now also C203.1
- net at C206.2, L202.2, U201.7 (OUTN): now also C204.1, RV202.1
- new net AGND: C201.2, C202.2, C203.2, C204.2, C207.1, C208.1, RV201.3, RV202.3, U201.15 (GND), U201.4 (GND), U201.5 (GND), U202.4 (OUTGND)
Changed lines of the file:
@@
-EESchema Schematic File Version 2  date Thu 28 Mar 2013 09:16:32 PM CET
+EESchema Schematic File Version 2  date Mon 01 Apr 2013 04:53:06 PM CEST
 LIBS:power
 LIBS:device
@@
 Sheet 2 6
 Title ""
-Date "28 mar 2013"
+Date "1 apr 2013"
 Rev ""
 Comp ""
@@
 $EndComp
 $Comp
-L GND #PWR019
-U 1 1 5151EC02
-P 6550 4400
-F 0 "#PWR019" H 6550 4400 30  0001 C CNN
-F 1 "GND" H 6550 4330 30  0001 C CNN
-F 2 "" H 6550 4400 60  0001 C CNN
-F 3 "" H 6550 4400 60  0001 C CNN
-	1    6550 4400
-	1    0    0    -1
-$EndComp
-$Comp
-L GND #PWR020
-U 1 1 5151EC1E
-P 5700 4250
-F 0 "#PWR020" H 5700 4250 30  0001 C CNN
-F 1 "GND" H 5700 4180 30  0001 C CNN
-F 2 "" H 5700 4250 60  0001 C CNN
-F 3 "" H 5700 4250 60  0001 C CNN
-	1    5700 4250
-	1    0    0    -1
-$EndComp
-$Comp
 L POT RV201
 U 1 1 5151EC34
@@
 	0    1    1    0
 $EndComp
-$Comp
-L GND #PWR021
-U 1 1 5151EC5D
-P 4800 3550
-F 0 "#PWR021" H 4800 3550 30  0001 C CNN
-F 1 "GND" H 4800 3480 30  0001 C CNN
-F 2 "" H 4800 3550 60  0001 C CNN
-F 3 "" H 4800 3550 60  0001 C CNN
-	1    4800 3550
-	1    0    0    -1
-$EndComp
 Text HLabel 6800 3400 2    60   Input ~ 0
 Enable
@@
 	7200 3500 6600 3500
 Wire Wire Line
-	6100 4350 5250 4350
+	6050 4350 5250 4350
 Wire Wire Line
 	5250 4350 5250 3900
@@
 	6800 3400 6600 3400
 Wire Wire Line
-	8050 3950 8050 3200
-Wire Wire Line
-	8050 3200 6600 3200
+	8050 3200 8050 3950
+Wire Wire Line
+	6600 3200 8050 3200
 Wire Wire Line
 	8050 4250 7550 4250
 Wire Wire Line
-	7550 3700 7550 4600
+	7550 4600 7550 3700
 Wire Wire Line
 	7550 3700 6600 3700
@@
 	5800 4200 5800 4600
 Connection ~ 5800 4600
-$Comp
-L GND #PWR022
-U 1 1 5151ED14
-P 7950 4150
-F 0 "#PWR022" H 7950 4150 30  0001 C CNN
-F 1 "GND" H 7950 4080 30  0001 C CNN
-F 2 "" H 7950 4150 60  0001 C CNN
-F 3 "" H 7950 4150 60  0001 C CNN
-	1    7950 4150
-	1    0    0    -1
-$EndComp
 Wire Wire Line
 	8050 4100 7950 4100
@@
 	1    0    0    -1
 $EndComp
-$Comp
-L GND #PWR023
-U 1 1 5151EE3B
-P 2900 3650
-F 0 "#PWR023" H 2900 3650 30  0001 C CNN
-F 1 "GND" H 2900 3580 30  0001 C CNN
-F 2 "" H 2900 3650 60  0001 C CNN
-F 3 "" H 2900 3650 60  0001 C CNN
-	1    2900 3650
-	1    0    0    -1
-$EndComp
-$Comp
-L GND #PWR024
-U 1 1 5151EE41
-P 2900 4300
-F 0 "#PWR024" H 2900 4300 30  0001 C CNN
-F 1 "GND" H 2900 4230 30  0001 C CNN
-F 2 "" H 2900 4300 60  0001 C CNN
-F 3 "" H 2900 4300 60  0001 C CNN
-	1    2900 4300
-	1    0    0    -1
-$EndComp
 Wire Wire Line
 	3150 3200 2900 3200
@@
 	-1   0    0    1
 $EndComp
-$Comp
-L GND #PWR025
-U 1 1 5151EEF5
-P 7000 5000
-F 0 "#PWR025" H 7000 5000 30  0001 C CNN
-F 1 "GND" H 7000 4930 30  0001 C CNN
-F 2 "" H 7000 5000 60  0001 C CNN
-F 3 "" H 7000 5000 60  0001 C CNN
-	1    7000 5000
-	1    0    0    -1
-$EndComp
-$Comp
-L GND #PWR026
-U 1 1 5151EEFB
-P 7800 3600
-F 0 "#PWR026" H 7800 3600 30  0001 C CNN
-F 1 "GND" H 7800 3530 30  0001 C CNN
-F 2 "" H 7800 3600 60  0001 C CNN
-F 3 "" H 7800 3600 60  0001 C CNN
-	1    7800 3600
-	1    0    0    -1
-$EndComp
-$Comp
-L GND #PWR027
-U 1 1 5151EF2F
-P 4550 3700
-F 0 "#PWR027" H 4550 3700 30  0001 C CNN
-F 1 "GND" H 4550 3630 30  0001 C CNN
-F 2 "" H 4550 3700 60  0001 C CNN
-F 3 "" H 4550 3700 60  0001 C CNN
-	1    4550 3700
-	1    0    0    -1
-$EndComp
 Wire Wire Line
 	5050 3500 5050 3600
@@
 -14
 $Comp
-L GND #PWR028
+L GND #PWR022
 U 1 1 5151EF8D
 P 7750 4500
-F 0 "#PWR028" H 7750 4500 30  0001 C CNN
+F 0 "#PWR022" H 7750 4500 30  0001 C CNN
 F 1 "GND" H 7750 4430 30  0001 C CNN
 F 2 "" H 7750 4500 60  0001 C CNN
@@
 	1    0    0    -1
 $EndComp
-$Comp
-L GND #PWR029
-U 1 1 5151F0CB
+Wire Wire Line
+	3900 3600 3900 3650
+Wire Wire Line
+	3900 4200 3900 4300
+Wire Wire Line
+	7800 3600 7800 3750
+Wire Wire Line
+	7000 5000 7000 5050
+Connection ~ 7800 3200
+Connection ~ 7000 4600
+$Comp
+L AGND #PWR023
+U 1 1 51584993
+P 7950 4150
+F 0 "#PWR023" H 7950 4150 40  0001 C CNN
+F 1 "AGND" H 7950 4080 50  0000 C CNN
+F 2 "" H 7950 4150 60  0000 C CNN
+F 3 "" H 7950 4150 60  0000 C CNN
+	1    7950 4150
+	1    0    0    -1
+$EndComp
+$Comp
+L AGND #PWR024
+U 1 1 515849A0
+P 7800 3750
+F 0 "#PWR024" H 7800 3750 40  0001 C CNN
+F 1 "AGND" H 7800 3680 50  0000 C CNN
+F 2 "" H 7800 3750 60  0000 C CNN
+F 3 "" H 7800 3750 60  0000 C CNN
+	1    7800 3750
+	1    0    0    -1
+$EndComp
+$Comp
+L AGND #PWR025
+U 1 1 515849B0
+P 7000 5050
+F 0 "#PWR025" H 7000 5050 40  0001 C CNN
+F 1 "AGND" H 7000 4980 50  0000 C CNN
+F 2 "" H 7000 5050 60  0000 C CNN
+F 3 "" H 7000 5050 60  0000 C CNN
+	1    7000 5050
+	1    0    0    -1
+$EndComp
+$Comp
+L AGND #PWR026
+U 1 1 515849B6
+P 6550 4400
+F 0 "#PWR026" H 6550 4400 40  0001 C CNN
+F 1 "AGND" H 6550 4330 50  0000 C CNN
+F 2 "" H 6550 4400 60  0000 C CNN
+F 3 "" H 6550 4400 60  0000 C CNN
+	1    6550 4400
+	1    0    0    -1
+$EndComp
+$Comp
+L AGND #PWR027
+U 1 1 515849BC
+P 5700 4250
+F 0 "#PWR027" H 5700 4250 40  0001 C CNN
+F 1 "AGND" H 5700 4180 50  0000 C CNN
+F 2 "" H 5700 4250 60  0000 C CNN
+F 3 "" H 5700 4250 60  0000 C CNN
+	1    5700 4250
+	1    0    0    -1
+$EndComp
+$Comp
+L AGND #PWR028
+U 1 1 515849C2
+P 4800 3650
+F 0 "#PWR028" H 4800 3650 40  0001 C CNN
+F 1 "AGND" H 4800 3580 50  0000 C CNN
+F 2 "" H 4800 3650 60  0000 C CNN
+F 3 "" H 4800 3650 60  0000 C CNN
+	1    4800 3650
+	1    0    0    -1
+$EndComp
+$Comp
+L AGND #PWR029
+U 1 1 515849CE
+P 4550 3700
+F 0 "#PWR029" H 4550 3700 40  0001 C CNN
+F 1 "AGND" H 4550 3630 50  0000 C CNN
+F 2 "" H 4550 3700 60  0000 C CNN
+F 3 "" H 4550 3700 60  0000 C CNN
+	1    4550 3700
+	1    0    0    -1
+$EndComp
+$Comp
+L AGND #PWR030
+U 1 1 515849D4
 P 3900 3650
-F 0 "#PWR029" H 3900 3650 30  0001 C CNN
-F 1 "GND" H 3900 3580 30  0001 C CNN
-F 2 "" H 3900 3650 60  0001 C CNN
-F 3 "" H 3900 3650 60  0001 C CNN
+F 0 "#PWR030" H 3900 3650 40  0001 C CNN
+F 1 "AGND" H 3900 3580 50  0000 C CNN
+F 2 "" H 3900 3650 60  0000 C CNN
+F 3 "" H 3900 3650 60  0000 C CNN
 	1    3900 3650
 	1    0    0    -1
 $EndComp
 $Comp
-L GND #PWR030
-U 1 1 5151F0D1
+L AGND #PWR031
+U 1 1 515849DA
 P 3900 4300
-F 0 "#PWR030" H 3900 4300 30  0001 C CNN
-F 1 "GND" H 3900 4230 30  0001 C CNN
-F 2 "" H 3900 4300 60  0001 C CNN
-F 3 "" H 3900 4300 60  0001 C CNN
+F 0 "#PWR031" H 3900 4300 40  0001 C CNN
+F 1 "AGND" H 3900 4230 50  0000 C CNN
+F 2 "" H 3900 4300 60  0000 C CNN
+F 3 "" H 3900 4300 60  0000 C CNN
 	1    3900 4300
 	1    0    0    -1
 $EndComp
-Wire Wire Line
-	3900 3600 3900 3650
-Wire Wire Line
-	3900 4200 3900 4300
+$Comp
+L AGND #PWR032
+U 1 1 515849E0
+P 2900 3650
+F 0 "#PWR032" H 2900 3650 40  0001 C CNN
+F 1 "AGND" H 2900 3580 50  0000 C CNN
+F 2 "" H 2900 3650 60  0000 C CNN
+F 3 "" H 2900 3650 60  0000 C CNN
+	1    2900 3650
+	1    0    0    -1
+$EndComp
+$Comp
+L AGND #PWR033
+U 1 1 515849E6
+P 2900 4300
+F 0 "#PWR033" H 2900 4300 40  0001 C CNN
+F 1 "AGND" H 2900 4230 50  0000 C CNN
+F 2 "" H 2900 4300 60  0000 C CNN
+F 3 "" H 2900 4300 60  0000 C CNN
+	1    2900 4300
+	1    0    0    -1
+$EndComp
+Text HLabel 7700 5050 0    60   Input ~ 0
+agnd
+$Comp
+L AGND #PWR034
+U 1 1 51584BC3
+P 7850 5100
+F 0 "#PWR034" H 7850 5100 40  0001 C CNN
+F 1 "AGND" H 7850 5030 50  0000 C CNN
+F 2 "" H 7850 5100 60  0000 C CNN
+F 3 "" H 7850 5100 60  0000 C CNN
+	1    7850 5100
+	1    0    0    -1
+$EndComp
+Wire Wire Line
+	7700 5050 7850 5050
+Wire Wire Line
+	7850 5050 7850 5100
+Wire Wire Line
+	4800 3550 4800 3650
+Connection ~ 3900 3200
+Connection ~ 3950 3800
+Connection ~ 2900 3200
+Connection ~ 2900 3800
+Connection ~ 3900 3800
 $EndSCHEMATC
