File: pcb/curry2.sch (KiCad schematic (older format))
At the start: 49 parts, among them CON101 AVR-ISP-6, IC101 ATMEGA88-A, P101 CONN_2, P102 CONN_4X2, SW101 SPST, SW102 SPST, U101 RASPI, U102 BQ32000, U103 ADS8568, X101 CRYSTAL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

Commit message: almost done
Parts:
- added R1: R, symbol R
Connections:
- net power/+5 is gone; now on net +5V: P101.1 (P1)
- net AGND: now also C104.2, C105.1, C106.2, C107.2, C108.1, C110.2, C111.2, C112.1, C117.2, C118.2, R1.1
- net GND: now also SW101.1, R1.2; no longer C117.2, C118.2
- net HVDD: now also C107.1, C111.1
- net HVSS: now also C108.2, C112.2
- net SCL: now also R102.2
- net SDA: now also R101.2
- net +5V: now reaches L102.1, L103.1, U101.2 (5V), U101.4 (5V)
- net at L103.2: now also L102.2, L104.2, L105.2
Other:
- moved on the sheet: X101

Commit message: almost done pre merger
Connections:
- net GND: no longer U101.35 (GND)
Changed lines of the file:
@@
-EESchema Schematic File Version 2  date Mon 01 Apr 2013 04:53:06 PM CEST
+EESchema Schematic File Version 2  date Tue 02 Apr 2013 02:33:42 PM CEST
 LIBS:power
 LIBS:device
@@
 Sheet 1 6
 Title ""
-Date "1 apr 2013"
+Date "2 apr 2013"
 Rev ""
 Comp ""
@@
 $EndComp
 $Comp
-L GND #PWR02
+L GND #PWR01
 U 1 1 51520228
 P 1050 1575
-F 0 "#PWR02" H 1050 1575 30  0001 C CNN
+F 0 "#PWR01" H 1050 1575 30  0001 C CNN
 F 1 "GND" H 1050 1505 30  0001 C CNN
 F 2 "" H 1050 1575 60  0001 C CNN
@@
 DVDD
 $Comp
-L GND #PWR03
+L GND #PWR02
 U 1 1 515208A0
 P 3400 2100
-F 0 "#PWR03" H 3400 2100 30  0001 C CNN
+F 0 "#PWR02" H 3400 2100 30  0001 C CNN
 F 1 "GND" H 3400 2030 30  0001 C CNN
 F 2 "" H 3400 2100 60  0001 C CNN
@@
 PAR
 $Comp
-L GND #PWR04
+L GND #PWR03
 U 1 1 51539576
 P 7950 6200
-F 0 "#PWR04" H 7950 6200 30  0001 C CNN
+F 0 "#PWR03" H 7950 6200 30  0001 C CNN
 F 1 "GND" H 7950 6130 30  0001 C CNN
 F 2 "" H 7950 6200 60  0001 C CNN
@@
 DVDD
 $Comp
-L GND #PWR05
+L GND #PWR04
 U 1 1 5153A199
 P 6500 5400
-F 0 "#PWR05" H 6500 5400 30  0001 C CNN
+F 0 "#PWR04" H 6500 5400 30  0001 C CNN
 F 1 "GND" H 6500 5330 30  0001 C CNN
 F 2 "" H 6500 5400 60  0001 C CNN
@@
 DVDD
 $Comp
-L GND #PWR06
+L GND #PWR05
 U 1 1 5153A6F5
 P 11150 4475
-F 0 "#PWR06" H 11150 4475 30  0001 C CNN
+F 0 "#PWR05" H 11150 4475 30  0001 C CNN
 F 1 "GND" H 11150 4405 30  0001 C CNN
 F 2 "" H 11150 4475 60  0001 C CNN
@@
 $Comp
 L GND #PWR07
-U 1 1 5153C3CF
-P 2900 4950
-F 0 "#PWR07" H 2900 4950 30  0001 C CNN
-F 1 "GND" H 2900 4880 30  0001 C CNN
-F 2 "" H 2900 4950 60  0001 C CNN
-F 3 "" H 2900 4950 60  0001 C CNN
-	1    2900 4950
-	1    0    0    -1
-$EndComp
-$Comp
-L GND #PWR08
 U 1 1 5153C605
 P 1950 4000
-F 0 "#PWR08" H 1950 4000 30  0001 C CNN
+F 0 "#PWR07" H 1950 4000 30  0001 C CNN
 F 1 "GND" H 1950 3930 30  0001 C CNN
 F 2 "" H 1950 4000 60  0001 C CNN
@@
 $EndComp
 $Comp
-L GND #PWR09
+L GND #PWR08
 U 1 1 5153C662
 P 4000 3950
-F 0 "#PWR09" H 4000 3950 30  0001 C CNN
+F 0 "#PWR08" H 4000 3950 30  0001 C CNN
 F 1 "GND" H 4000 3880 30  0001 C CNN
 F 2 "" H 4000 3950 60  0001 C CNN
@@
 $EndComp
 $Comp
-L GND #PWR010
+L GND #PWR09
 U 1 1 5153DB5A
 P 3650 2525
-F 0 "#PWR010" H 3650 2525 30  0001 C CNN
+F 0 "#PWR09" H 3650 2525 30  0001 C CNN
 F 1 "GND" H 3650 2455 30  0001 C CNN
 F 2 "" H 3650 2525 60  0001 C CNN
@@
 $EndComp
 $Comp
-L GND #PWR011
+L GND #PWR010
 U 1 1 5153DBB7
 P 3675 2850
-F 0 "#PWR011" H 3675 2850 30  0001 C CNN
+F 0 "#PWR010" H 3675 2850 30  0001 C CNN
 F 1 "GND" H 3675 2780 30  0001 C CNN
 F 2 "" H 3675 2850 60  0001 C CNN
@@
 $EndComp
 $Comp
-L GND #PWR012
+L GND #PWR011
 U 1 1 5153DEDE
 P 1750 3225
-F 0 "#PWR012" H 1750 3225 30  0001 C CNN
+F 0 "#PWR011" H 1750 3225 30  0001 C CNN
 F 1 "GND" H 1750 3155 30  0001 C CNN
 F 2 "" H 1750 3225 60  0001 C CNN
@@
 DVDD
 $Comp
-L GND #PWR013
+L GND #PWR012
 U 1 1 5154260A
 P 3525 6025
-F 0 "#PWR013" H 3525 6025 30  0001 C CNN
+F 0 "#PWR012" H 3525 6025 30  0001 C CNN
 F 1 "GND" H 3525 5955 30  0001 C CNN
 F 2 "" H 3525 6025 60  0001 C CNN
@@
 SCL
 $Comp
-L GND #PWR014
+L GND #PWR013
 U 1 1 51543461
 P 3975 7400
-F 0 "#PWR014" H 3975 7400 30  0001 C CNN
+F 0 "#PWR013" H 3975 7400 30  0001 C CNN
 F 1 "GND" H 3975 7330 30  0001 C CNN
 F 2 "" H 3975 7400 60  0001 C CNN
@@
 $EndComp
 $Comp
-L GND #PWR015
+L GND #PWR014
 U 1 1 515445A2
 P 4675 5925
-F 0 "#PWR015" H 4675 5925 30  0001 C CNN
+F 0 "#PWR014" H 4675 5925 30  0001 C CNN
 F 1 "GND" H 4675 5855 30  0001 C CNN
 F 2 "" H 4675 5925 60  0001 C CNN
@@
 $EndComp
 $Comp
-L GND #PWR016
+L GND #PWR015
 U 1 1 5154C56D
 P 8675 5275
-F 0 "#PWR016" H 8675 5275 30  0001 C CNN
+F 0 "#PWR015" H 8675 5275 30  0001 C CNN
 F 1 "GND" H 8675 5205 30  0001 C CNN
 F 2 "" H 8675 5275 60  0001 C CNN
@@
 $EndComp
 $Comp
-L GND #PWR017
+L GND #PWR016
 U 1 1 5154CC74
 P 9100 7125
-F 0 "#PWR017" H 9100 7125 30  0001 C CNN
+F 0 "#PWR016" H 9100 7125 30  0001 C CNN
 F 1 "GND" H 9100 7055 30  0001 C CNN
 F 2 "" H 9100 7125 60  0001 C CNN
@@
 $EndComp
 $Comp
-L GND #PWR018
+L GND #PWR017
 U 1 1 5154D766
 P 5625 7425
-F 0 "#PWR018" H 5625 7425 30  0001 C CNN
+F 0 "#PWR017" H 5625 7425 30  0001 C CNN
 F 1 "GND" H 5625 7355 30  0001 C CNN
 F 2 "" H 5625 7425 60  0001 C CNN
@@
 $EndComp
 $Comp
-L GND #PWR019
+L GND #PWR018
 U 1 1 51586021
 P 2800 5250
-F 0 "#PWR019" H 2800 5250 30  0001 C CNN
+F 0 "#PWR018" H 2800 5250 30  0001 C CNN
 F 1 "GND" H 2800 5180 30  0001 C CNN
 F 2 "" H 2800 5250 60  0001 C CNN
@@
 $EndComp
 $Comp
-L +5V #PWR020
+L +5V #PWR019
 U 1 1 5158CA84
 P 3300 1950
-F 0 "#PWR020" H 3300 2040 20  0001 C CNN
+F 0 "#PWR019" H 3300 2040 20  0001 C CNN
 F 1 "+5V" H 3300 2040 30  0000 C CNN
 F 2 "" H 3300 1950 60  0000 C CNN
@@
 $EndComp
 $Comp
-L +5V #PWR021
+L +5V #PWR020
 U 1 1 5158CF7D
 P 7750 6350
-F 0 "#PWR021" H 7750 6440 20  0001 C CNN
+F 0 "#PWR020" H 7750 6440 20  0001 C CNN
 F 1 "+5V" H 7750 6440 30  0000 C CNN
 F 2 "" H 7750 6350 60  0000 C CNN
@@
 	8375 4050 8375 3975
 Wire Wire Line
-	2900 4500 2900 4950
-Wire Wire Line
 	4000 3850 4000 3950
