File: pcb/curry2.sch (KiCad schematic (older format))
At the start: 50 parts, among them CON101 AVR-ISP-6, IC101 ATMEGA88-A, P101 CONN_2, P102 CONN_4X2, SW101 SPST, SW102 SPST, U101 RASPI, U102 BQ32000, U103 ADS8568, X101 CRYSTAL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

Commit message: städa lite
Parts:
- R1: value R -> 0R?
- X101: value CRYSTAL -> 32K768
Connections:
- net AGND: now also R1.2; no longer R1.1
- net GND: now also IC101.21 (GND), IC101.5 (GND), R1.1; no longer R1.2
- net at IC101.11 ((PCINT23/AIN1)PD7), P102.2, P102.8: now also P102.4, P102.6
- net power/Enable renamed PWEN
Other:
- moved on the sheet: BT101, C103, C104, C105, C106, C107, C108, C109, C110, C111, C112, C113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

Commit message: fuffens
Parts:
- R102: value R -> 4k7
Connections:
- net CS: now also U101.31 (GPIO30)
- net DVDD: now also R102.2; no longer R102.1
- net GND: now also U101.33 (GND), U101.34 (GND), U101.36 (GND), U101.37 (GND), U101.38 (GND)
- net SCL: now also R102.1, U101.30 (GPIO29); no longer R102.2
- net SDA: now also U101.29 (GPIO28)
Other:
- moved on the sheet: P101, R101, R102

Commit message: wip
Connections:
- net GND: no longer U101.35 (GND), U101.36 (GND), U101.37 (GND), U101.38 (GND)
Changed lines of the file:
@@
-EESchema Schematic File Version 2  date Tue 02 Apr 2013 03:24:17 PM CEST
+EESchema Schematic File Version 2  date Tue 02 Apr 2013 03:29:12 PM CEST
 LIBS:power
 LIBS:device
@@
 $EndComp
 $Comp
-L GND #PWR07
-U 1 1 5153C3CF
-P 3300 4200
-F 0 "#PWR07" H 3300 4200 30  0001 C CNN
-F 1 "GND" H 3300 4130 30  0001 C CNN
-F 2 "" H 3300 4200 60  0001 C CNN
-F 3 "" H 3300 4200 60  0001 C CNN
-	1    3300 4200
-	1    0    0    -1
-$EndComp
-$Comp
 L GND #PWR08
 U 1 1 5153C605
@@
 Wire Wire Line
 	1850 3700 1850 3800
-$Comp
-L GND #PWR?
-U 1 1 515B25BC
-P 1850 4200
-F 0 "#PWR?" H 1850 4200 30  0001 C CNN
-F 1 "GND" H 1850 4130 30  0001 C CNN
-F 2 "" H 1850 4200 60  0001 C CNN
-F 3 "" H 1850 4200 60  0001 C CNN
-	1    1850 4200
-	1    0    0    -1
-$EndComp
-Wire Wire Line
-	1850 4000 1850 4100
-Wire Wire Line
-	1850 4100 1850 4200
-Wire Wire Line
-	1850 4000 1950 4000
-Wire Wire Line
-	1950 4100 1850 4100
-Connection ~ 1850 4100
-Wire Wire Line
-	3300 4000 3300 4100
-Wire Wire Line
-	3300 4100 3300 4200
-Wire Wire Line
-	3300 4000 3200 4000
-Wire Wire Line
-	3200 4100 3300 4100
-Connection ~ 3300 4100
 Wire Wire Line
 	1850 3300 1850 3500

Commit message: pcb done just needs currentsensors
Parts:
- removed BT101: BATTERY, symbol BATTERY
- removed X101: 32K768, symbol CRYSTAL
- added P1, P2: CONN_4, symbol CONN_4
Connections:
- net +5V: now also P1.4 (P4)
- net DB10: now also U101.19 (GPIO10); no longer U101.18 (GPIO24)
- net DB11: now also U101.21 (GPIO9); no longer U101.19 (GPIO10)
- net DB12: now also U101.22 (GPIO25); no longer U101.21 (GPIO9)
- net DB13: now also U101.24 (GPIO8); no longer U101.22 (GPIO25)
- net DB15: now also U101.26 (GPIO7); no longer U101.24 (GPIO8)
- net DB3: now also U101.10 (GPIO15); no longer U101.9 (GND)
- net DB4: now also U101.11 (GPIO17); no longer U101.10 (GPIO15)
- net DB5: now also U101.12 (GPIO18); no longer U101.11 (GPIO17)
- net DB6: now also U101.13 (GPIO27); no longer U101.12 (GPIO18)
- net DB7: now also U101.15 (GPIO22); no longer U101.13 (GPIO27)
- net DB8: now also U101.16 (GPIO23); no longer U101.15 (GPIO22)
- net DB9: now also U101.18 (GPIO24); no longer U101.16 (GPIO23)
- net GND: now also U101.9 (GND), P1.1 (P1), P2.1 (P1)
- net RD: now also U101.32 (GPIO31); no longer U101.26 (GPIO7)
- net SCL: now also P1.2 (P2)
- net SDA: now also P1.3 (P3)
- net at IC101.10 ((PCINT22/OC0A/AIN0)PD6): now also P102.2, P102.4, P102.6, P102.8
- net at U102.1 (OSCI): now also P2.3 (P3)
- net at U102.2 (OSCO): now also P2.4 (P4)
- net at U102.3 (VBAT): now also P2.2 (P2)
- now unconnected: IC101.11 ((PCINT23/AIN1)PD7)
